File: schematic/schematic.kicad_sch (KiCad schematic)
At the start: 6 parts, among them SW1 CK_KMS2xxGP, SW2 CK_KMS2xxGP, U3 ESP32-WROOM-32

Commit message: ++ Introduction chapter ++ doxygen +- Main part
Other:
- note removed: "Buttons"
- moved on the sheet: DS1, R1, R2, SW1, SW2, U3
